Commit message: aansturingv1.4
Robot arm begint straight op. Robot arm heeft nu ook servo restricties geimplementeerd. Op het moment bezig dat de single servo aansturing real-time gebeurt. Als dit lukt dan wordt dit ook gedaan voor group command. Op dit moment verplaats van de arm van punt A naar B in een keer.

File: src/robot_arm_simulatie_bp/urdf/lynxmotion_arm.urdf (robot description, URDF)
Before this commit: robot lynxmotion_arm, 8 links, 7 joints
Joints:
- joint upperarm2forearm: origin xyz=0 0 0.18 rpy=0 1.5708 0 -> xyz=0 0 0.18 rpy=0 0 0
